File: ICBlockBusPcb.kicad_pcb (KiCad board)
At the start: 2 copper layers, 204.5 x 20.3 mm, 61 parts, among them J1 Conn_01x04_Pin, J10 Conn_01x06_Pin, J11 Conn_01x06_Socket, J12 Conn_01x06_Pin, J13 Conn_01x06_Socket, J14 Conn_01x06_Pin, J15 Conn_01x06_Socket, J16 Conn_01x06_Pin, J17 Conn_01x06_Socket, J18 Conn_01x06_Pin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

Commit message: rev 1.2 prod
Parts:
- added FID1: Fiducial, Fiducial:Fiducial_0.5mm_Mask1mm, F.Cu at (61.0, 109.2)
- added FID2: Fiducial, Fiducial:Fiducial_0.5mm_Mask1mm, B.Cu at (61.0, 109.2)
- added H1: MountingHole, MountingHole:MountingHole_2.2mm_M2, F.Cu at (61.0, 97.8)
- added H2: MountingHole, MountingHole:MountingHole_2.2mm_M2, F.Cu at (195.6, 108.0)
- added H3: MountingHole, MountingHole:MountingHole_2.2mm_M2, F.Cu at (222.9, 97.8)
- added H4: MountingHole, MountingHole:MountingHole_2.2mm_M2, F.Cu at (87.6, 108.0)
- moved C1 29.2 mm to (170.8, 95.9), turned to 0 degrees
Connections:
- J10 pad 1: unconnected-(J10-Pin_1-Pad1) -> Net-(J10-Pin_1)
- J10 pad 6: unconnected-(J10-Pin_6-Pad6) -> Net-(J10-Pin_6)
- J11 pad 1: unconnected-(J11-Pin_1-Pad1) -> Net-(J11-Pin_1)
- J11 pad 6: unconnected-(J11-Pin_6-Pad6) -> Net-(J11-Pin_6)
- J12 pad 1: unconnected-(J12-Pin_1-Pad1) -> Net-(J11-Pin_1)
- J12 pad 6: unconnected-(J12-Pin_6-Pad6) -> Net-(J11-Pin_6)
- J13 pad 1: unconnected-(J13-Pin_1-Pad1) -> Net-(J13-Pin_1)
- J13 pad 6: unconnected-(J13-Pin_6-Pad6) -> Net-(J13-Pin_6)
- J14 pad 1: unconnected-(J14-Pin_1-Pad1) -> Net-(J13-Pin_1)
- J14 pad 6: unconnected-(J14-Pin_6-Pad6) -> Net-(J13-Pin_6)
- J15 pad 1: unconnected-(J15-Pin_1-Pad1) -> Net-(J15-Pin_1)
- J15 pad 6: unconnected-(J15-Pin_6-Pad6) -> Net-(J15-Pin_6)
- J16 pad 1: unconnected-(J16-Pin_1-Pad1) -> Net-(J15-Pin_1)
- J16 pad 6: unconnected-(J16-Pin_6-Pad6) -> Net-(J15-Pin_6)
- J17 pad 1: unconnected-(J17-Pin_1-Pad1) -> Net-(J17-Pin_1)
- J17 pad 6: unconnected-(J17-Pin_6-Pad6) -> Net-(J17-Pin_6)
- J18 pad 1: unconnected-(J18-Pin_1-Pad1) -> Net-(J17-Pin_1)
- J18 pad 6: unconnected-(J18-Pin_6-Pad6) -> Net-(J17-Pin_6)
- J3 pad 1: unconnected-(J3-Pin_1-Pad1) -> Net-(J3-Pin_1)
- J3 pad 6: unconnected-(J3-Pin_6-Pad6) -> Net-(J3-Pin_6)
- J4 pad 1: unconnected-(J4-Pin_1-Pad1) -> Net-(J3-Pin_1)
- J4 pad 6: unconnected-(J4-Pin_6-Pad6) -> Net-(J3-Pin_6)
- J5 pad 1: unconnected-(J5-Pin_1-Pad1) -> Net-(J5-Pin_1)
- J5 pad 6: unconnected-(J5-Pin_6-Pad6) -> Net-(J5-Pin_6)
- J6 pad 1: unconnected-(J6-Pin_1-Pad1) -> Net-(J5-Pin_1)
- J6 pad 6: unconnected-(J6-Pin_6-Pad6) -> Net-(J5-Pin_6)
- J7 pad 1: unconnected-(J7-Pin_1-Pad1) -> Net-(J7-Pin_1)
- J7 pad 6: unconnected-(J7-Pin_6-Pad6) -> Net-(J7-Pin_6)
- J8 pad 1: unconnected-(J8-Pin_1-Pad1) -> Net-(J7-Pin_1)
- J8 pad 6: unconnected-(J8-Pin_6-Pad6) -> Net-(J7-Pin_6)
- J9 pad 1: unconnected-(J9-Pin_1-Pad1) -> Net-(J10-Pin_1)
- J9 pad 6: unconnected-(J9-Pin_6-Pad6) -> Net-(J10-Pin_6)
Routing:
- net Net-(J11-Pin_6): track 0.00 -> 35.0 mm, vias 0 -> 1
- net Net-(J7-Pin_6): track 0.00 -> 12.7 mm
- net Net-(J7-Pin_1): track 0.00 -> 12.7 mm
- net Net-(J5-Pin_6): track 0.00 -> 12.7 mm
- net Net-(J5-Pin_1): track 0.00 -> 12.7 mm
- net Net-(J3-Pin_6): track 0.00 -> 12.7 mm
- net Net-(J3-Pin_1): track 0.00 -> 12.7 mm
- net Net-(J17-Pin_6): track 0.00 -> 12.7 mm
- net Net-(J17-Pin_1): track 0.00 -> 12.7 mm
- net Net-(J15-Pin_6): track 0.00 -> 12.7 mm
- net Net-(J15-Pin_1): track 0.00 -> 12.7 mm
- net Net-(J13-Pin_6): track 0.00 -> 12.7 mm
- net Net-(J13-Pin_1): track 0.00 -> 12.7 mm
- net Net-(J10-Pin_6): track 0.00 -> 12.7 mm
- net Net-(J10-Pin_1): track 0.00 -> 12.7 mm
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- added copper zone on B.Cu, net VCC
Other:
- outline, holes or cut-outs redrawn
- board text added: "BOTTOM"
- board text added: "GL"
- board text added: "GR"
- board text added: "INPUT"
- board text added: "OUTPUT"
- board text added: "RL"
- board text added: "RR"
- board text added: "TCA9548A"
- board text added: "TOP"
