File: ICBlockBusPcb.kicad_sch (KiCad schematic)
At the start: 61 parts, among them J1 Conn_01x04_Pin, J10 Conn_01x06_Pin, J11 Conn_01x06_Socket, J12 Conn_01x06_Pin, J13 Conn_01x06_Socket, J14 Conn_01x06_Pin, J15 Conn_01x06_Socket, J16 Conn_01x06_Pin, J17 Conn_01x06_Socket, J18 Conn_01x06_Pin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

Commit message: rev 1.2 prod
Parts:
- added FID1, FID2: Fiducial, Fiducial:Fiducial_0.5mm_Mask1mm, symbol Mechanical:Fiducial
- added H1, H2, H3, H4: MountingHole, MountingHole:MountingHole_2.2mm_M2, symbol Mechanical:MountingHole
Connections:
- net at J17.1 (Pin_1): now also J18.1 (Pin_1)
- net at J17.6 (Pin_6): now also J18.6 (Pin_6)
- net at J11.1 (Pin_1): now also J12.1 (Pin_1)
- net at J11.6 (Pin_6): now also J12.6 (Pin_6)
- net at J13.1 (Pin_1): now also J14.1 (Pin_1)
- net at J13.6 (Pin_6): now also J14.6 (Pin_6)
- net at J8.1 (Pin_1): now also J7.1 (Pin_1)
- net at J8.6 (Pin_6): now also J7.6 (Pin_6)
- net at J3.1 (Pin_1): now also J4.1 (Pin_1)
- net at J3.6 (Pin_6): now also J4.6 (Pin_6)
- net at J6.1 (Pin_1): now also J5.1 (Pin_1)
- net at J6.6 (Pin_6): now also J5.6 (Pin_6)
- net at J16.1 (Pin_1): now also J15.1 (Pin_1)
- net at J16.6 (Pin_6): now also J15.6 (Pin_6)
- net at J9.1 (Pin_1): now also J10.1 (Pin_1)
- net at J9.6 (Pin_6): now also J10.6 (Pin_6)
- no-connect marks 32 -> 0
Other:
- moved on the sheet: J10, J11, J12, J13, J14, J15, J16, J17, J18, J3, J4, J5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
